File: dvi-12bit/v1.1b-1c/dvi-12bit.kicad_pcb (KiCad board)
At the start: 4 copper layers, 43.6 x 34 mm, 29 parts, among them J1 Conn_02x10_Odd_Even, J10 sj, J6 HDMI_A_1.4, J7 sj, J8 sj, J9 sj, U2 SII164

Commit message: Version 0.1
Parts:
- J6: footprint pkl_connectors:HDMI-10029449-111RLF -> custom:HDMI-SMD_HDMI-001S
- moved J6 2.73 mm to (68.6, 39.4)
Routing:
- net GND: track 43.4 -> 36.5 mm
- net +3V3: track 15.1 -> 15.8 mm
Other:
- board size 43.6 x 34 mm -> 45.6 x 34 mm
- board text added: "HDMI EXT CARD(24b) Ver0.1"
