File: dvi-12bit/v1.1b-1c/dvi-12bit.kicad_sch (KiCad schematic)
At the start: 29 parts, among them J1 Conn_02x10_Odd_Even, J10 sj, J6 HDMI_A_1.4, J7 sj, J8 sj, J9 sj, U2 SII164

Commit message: Version 0.1
Parts:
- J6: footprint pkl_connectors:HDMI-10029449-111RLF -> custom:HDMI-SMD_HDMI-001S
Changed lines of the file:
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@@
     (effects (font (size 1.27 1.27)) (justify right bottom))
   )
-  (label "TVDD" (at 190.5 99.06 0)
+  (label "TVDD" (at 190.5 99.06 0) (fields_autoplaced)
     (effects (font (size 1.27 1.27)) (justify left bottom))
   )
-  (label "B2" (at 142.24 99.06 180)
+  (label "B2" (at 142.24 99.06 180) (fields_autoplaced)
     (effects (font (size 1.27 1.27)) (justify right bottom))
   )
-  (label "DK3" (at 142.24 134.62 180)
+  (label "DK3" (at 142.24 134.62 180) (fields_autoplaced)
     (effects (font (size 1.27 1.27)) (justify right bottom))
   )
-  (label "CK-" (at 200.66 78.74 0)
+  (label "CK-" (at 200.66 78.74 0) (fields_autoplaced)
     (effects (font (size 1.27 1.27)) (justify left bottom))
   )
-  (label "D0+" (at 243.84 83.82 180)
+  (label "D0+" (at 243.84 83.82 180) (fields_autoplaced)
     (effects (font (size 1.27 1.27)) (justify right bottom))
   )
-  (label "VREF" (at 142.24 116.84 180)
+  (label "VREF" (at 142.24 116.84 180) (fields_autoplaced)
     (effects (font (size 1.27 1.27)) (justify right bottom))
   )
-  (label "D2-" (at 243.84 76.2 180)
+  (label "D2-" (at 243.84 76.2 180) (fields_autoplaced)
     (effects (font (size 1.27 1.27)) (justify right bottom))
   )
-  (label "D1+" (at 200.66 66.04 0)
+  (label "D1+" (at 200.66 66.04 0) (fields_autoplaced)
     (effects (font (size 1.27 1.27)) (justify left bottom))
   )
@@
     (effects (font (size 1.27 1.27)) (justify left bottom))
   )
-  (label "B0" (at 142.24 104.14 180)
+  (label "B0" (at 142.24 104.14 180) (fields_autoplaced)
     (effects (font (size 1.27 1.27)) (justify right bottom))
   )
-  (label "D2+" (at 200.66 71.12 0)
+  (label "D2+" (at 200.66 71.12 0) (fields_autoplaced)
     (effects (font (size 1.27 1.27)) (justify left bottom))
   )
-  (label "G3" (at 142.24 86.36 180)
+  (label "G3" (at 142.24 86.36 180) (fields_autoplaced)
     (effects (font (size 1.27 1.27)) (justify right bottom))
   )
-  (label "R3" (at 142.24 76.2 180)
+  (label "R3" (at 142.24 76.2 180) (fields_autoplaced)
     (effects (font (size 1.27 1.27)) (justify right bottom))
   )
-  (label "DK2" (at 142.24 137.16 180)
+  (label "DK2" (at 142.24 137.16 180) (fields_autoplaced)
     (effects (font (size 1.27 1.27)) (justify right bottom))
   )
-  (label "~{PD}" (at 142.24 129.54 180)
+  (label "~{PD}" (at 142.24 129.54 180) (fields_autoplaced)
     (effects (font (size 1.27 1.27)) (justify right bottom))
   )
-  (label "D2+" (at 243.84 73.66 180)
+  (label "D2+" (at 243.84 73.66 180) (fields_autoplaced)
     (effects (font (size 1.27 1.27)) (justify right bottom))
   )
-  (label "B3" (at 142.24 96.52 180)
+  (label "B3" (at 142.24 96.52 180) (fields_autoplaced)
     (effects (font (size 1.27 1.27)) (justify right bottom))
   )
@@
     (effects (font (size 1.27 1.27)) (justify right bottom))
   )
-  (label "CLK" (at 142.24 40.64 180)
+  (label "CLK" (at 142.24 40.64 180) (fields_autoplaced)
     (effects (font (size 1.27 1.27)) (justify right bottom))
   )
-  (label "CK+" (at 200.66 76.2 0)
+  (label "CK+" (at 200.66 76.2 0) (fields_autoplaced)
     (effects (font (size 1.27 1.27)) (justify left bottom))
   )
-  (label "D2-" (at 200.66 73.66 0)
+  (label "D2-" (at 200.66 73.66 0) (fields_autoplaced)
     (effects (font (size 1.27 1.27)) (justify left bottom))
   )
@@
     (effects (font (size 1.27 1.27)) (justify left bottom))
   )
-  (label "D0-" (at 200.66 63.5 0)
+  (label "D0-" (at 200.66 63.5 0) (fields_autoplaced)
     (effects (font (size 1.27 1.27)) (justify left bottom))
   )
-  (label "R0" (at 142.24 83.82 180)
+  (label "R0" (at 142.24 83.82 180) (fields_autoplaced)
     (effects (font (size 1.27 1.27)) (justify right bottom))
   )
-  (label "D0-" (at 243.84 86.36 180)
+  (label "D0-" (at 243.84 86.36 180) (fields_autoplaced)
     (effects (font (size 1.27 1.27)) (justify right bottom))
   )
@@
     (effects (font (size 1.27 1.27)) (justify right bottom))
   )
-  (label "D0+" (at 200.66 60.96 0)
+  (label "D0+" (at 200.66 60.96 0) (fields_autoplaced)
     (effects (font (size 1.27 1.27)) (justify left bottom))
   )
@@
     (effects (font (size 1.27 1.27)) (justify left bottom))
   )
-  (label "DE" (at 142.24 109.22 180)
+  (label "DE" (at 142.24 109.22 180) (fields_autoplaced)
     (effects (font (size 1.27 1.27)) (justify right bottom))
   )
-  (label "DSEL-SDA" (at 142.24 147.32 180)
+  (label "DSEL-SDA" (at 142.24 147.32 180) (fields_autoplaced)
     (effects (font (size 1.27 1.27)) (justify right bottom))
   )
-  (label "PVCC" (at 190.5 93.98 0)
+  (label "PVCC" (at 190.5 93.98 0) (fields_autoplaced)
     (effects (font (size 1.27 1.27)) (justify left bottom))
   )
-  (label "D1-" (at 243.84 81.28 180)
+  (label "D1-" (at 243.84 81.28 180) (fields_autoplaced)
     (effects (font (size 1.27 1.27)) (justify right bottom))
   )
-  (label "VCC" (at 190.5 86.36 0)
+  (label "VCC" (at 190.5 86.36 0) (fields_autoplaced)
     (effects (font (size 1.27 1.27)) (justify left bottom))
   )
-  (label "TFADJ" (at 193.04 81.28 0)
+  (label "TFADJ" (at 193.04 81.28 0) (fields_autoplaced)
     (effects (font (size 1.27 1.27)) (justify left bottom))
   )
@@
     (effects (font (size 1.27 1.27)) (justify right bottom))
   )
-  (label "CK+" (at 243.84 88.9 180)
+  (label "CK+" (at 243.84 88.9 180) (fields_autoplaced)
     (effects (font (size 1.27 1.27)) (justify right bottom))
   )
-  (label "EDGE-HTPLG" (at 142.24 119.38 180)
+  (label "EDGE-HTPLG" (at 142.24 119.38 180) (fields_autoplaced)
     (effects (font (size 1.27 1.27)) (justify right bottom))
   )
-  (label "BSEL-SCL" (at 142.24 144.78 180)
+  (label "BSEL-SCL" (at 142.24 144.78 180) (fields_autoplaced)
     (effects (font (size 1.27 1.27)) (justify right bottom))
   )
-  (label "DKEN" (at 142.24 121.92 180)
+  (label "DKEN" (at 142.24 121.92 180) (fields_autoplaced)
     (effects (font (size 1.27 1.27)) (justify right bottom))
   )
-  (label "R1" (at 142.24 81.28 180)
+  (label "R1" (at 142.24 81.28 180) (fields_autoplaced)
     (effects (font (size 1.27 1.27)) (justify right bottom))
   )
@@
     (effects (font (size 1.27 1.27)) (justify right bottom))
   )
-  (label "HS" (at 142.24 114.3 180)
+  (label "HS" (at 142.24 114.3 180) (fields_autoplaced)
     (effects (font (size 1.27 1.27)) (justify right bottom))
   )
-  (label "G2" (at 142.24 88.9 180)
+  (label "G2" (at 142.24 88.9 180) (fields_autoplaced)
     (effects (font (size 1.27 1.27)) (justify right bottom))
   )
@@
     (effects (font (size 1.27 1.27)) (justify left bottom))
   )
-  (label "CK-" (at 243.84 91.44 180)
+  (label "CK-" (at 243.84 91.44 180) (fields_autoplaced)
     (effects (font (size 1.27 1.27)) (justify right bottom))
   )
@@
     (effects (font (size 1.27 1.27)) (justify left bottom))
   )
-  (label "D1-" (at 200.66 68.58 0)
+  (label "D1-" (at 200.66 68.58 0) (fields_autoplaced)
     (effects (font (size 1.27 1.27)) (justify left bottom))
   )
-  (label "R2" (at 142.24 78.74 180)
+  (label "R2" (at 142.24 78.74 180) (fields_autoplaced)
     (effects (font (size 1.27 1.27)) (justify right bottom))
   )
@@
     (effects (font (size 1.27 1.27)) (justify right bottom))
   )
-  (label "B1" (at 142.24 101.6 180)
+  (label "B1" (at 142.24 101.6 180) (fields_autoplaced)
     (effects (font (size 1.27 1.27)) (justify right bottom))
   )
-  (label "G0" (at 142.24 93.98 180)
+  (label "G0" (at 142.24 93.98 180) (fields_autoplaced)
     (effects (font (size 1.27 1.27)) (justify right bottom))
   )
@@
     (effects (font (size 1.27 1.27)) (justify left bottom))
   )
-  (label "G1" (at 142.24 91.44 180)
+  (label "G1" (at 142.24 91.44 180) (fields_autoplaced)
     (effects (font (size 1.27 1.27)) (justify right bottom))
   )
-  (label "DK1" (at 142.24 139.7 180)
+  (label "DK1" (at 142.24 139.7 180) (fields_autoplaced)
     (effects (font (size 1.27 1.27)) (justify right bottom))
   )
-  (label "VS" (at 142.24 111.76 180)
+  (label "VS" (at 142.24 111.76 180) (fields_autoplaced)
     (effects (font (size 1.27 1.27)) (justify right bottom))
   )
-  (label "D1+" (at 243.84 78.74 180)
+  (label "D1+" (at 243.84 78.74 180) (fields_autoplaced)
     (effects (font (size 1.27 1.27)) (justify right bottom))
   )
-  (label "ISEL-~{RST}" (at 142.24 132.08 180)
+  (label "ISEL-~{RST}" (at 142.24 132.08 180) (fields_autoplaced)
     (effects (font (size 1.27 1.27)) (justify right bottom))
   )
@@
       (effects (font (size 1.27 1.27)) (justify left))
     )
-    (property "Footprint" "pkl_connectors:HDMI-10029449-111RLF" (at 257.175 93.98 0)
+    (property "Footprint" "custom:HDMI-SMD_HDMI-001S" (at 257.175 93.98 0)
       (effects (font (size 1.27 1.27)) hide)
     )
